File: connector_board.kicad_sch (KiCad schematic)
At the start: 2 parts, among them J1 Screw Terminal Block 5.00 mm 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

Commit message: feat: add connectors
Parts:
- removed R1: 47k_0805, Resistor_SMD:R_0805_2012Metric, symbol 2s_Resistor_0805:47k_0805
- added H1, H2, H3, H4: MountingHole, MountingHole:MountingHole_3.2mm_M3_Pad, symbol Mechanical:MountingHole
- added J10: Screw Terminal Block 3.50 mm 2 pol, 2s_connectors:TerminalBlock_4Ucon_1x02_P3.50mm_Horizontal, symbol 2s_connectors:1751248
- added J11: 2s-tc2030-NL, Connector:Tag-Connect_TC2030-IDC-NL_2x03_P1.27mm_Vertical, symbol 2s_connectors:2s_tag_connect_6 NL
- added J12: TC2050 With UART NL, Connector:Tag-Connect_TC2050-IDC-NL_2x05_P1.27mm_Vertical, symbol 2s_connectors:2s_tag_connect_10 NL
- added J2: 2s_cortex-m-10-pin, 2s_connectors:PinHeader_2x5_P1.27_SMD, symbol 2s_connectors:2s_cortex-m-10-pin
- added J3: 2s-tc2030, Connector:Tag-Connect_TC2030-IDC-FP_2x03_P1.27mm_Vertical, symbol 2s_connectors:2s_tag_connect_6
- added J4: 2s_cortex-m-10-pin, Connector:Tag-Connect_TC2050-IDC-FP_2x05_P1.27mm_Vertical, symbol 2s_connectors:2s_tag_connect_10
- added J5: 1757242, Connector_Phoenix_MSTB:PhoenixContact_MSTBA_2,5_2-G-5,08_1x02_P5.08mm_Horizontal, symbol 2s_connectors:1757242
- added J6: S3B-ZR-SM4A-TF, 2s_connectors:JST_ZH_B3B-ZR-SM4-TF_1x03-1MP_P1.50mm_Vertical, symbol 2s_connectors:JST S3B-ZR-SM4A-TF
- added J7: JST S3B-XH-A, Connector_JST:JST_XH_S3B-XH-A_1x03_P2.50mm_Horizontal, symbol 2s_connectors:JST S3B-XH-A
- added J8: JST S3B-PH-K-S, Connector_JST:JST_PH_S3B-PH-K_1x03_P2.00mm_Horizontal, symbol 2s_connectors:JST S3B-PH-K-S
- added J9: JST SM03B-SRSS-TB, 2s_connectors:JST_SH_SM03B-SRSS-TB_1x03-1MP_P1.00mm_Horizontal, symbol 2s_connectors:JST SM03B-SRSS-TB
Connections:
- net GND: no longer names the net of J1.1 (Pin_1)
- no-connect marks 0 -> 60

Commit message: feat: even more connectors
BREAKING CHANGE:
Parts:
- added J13: 1-350942-0, 2s_connectors:CONN_1-350942-0_TYC, symbol 2s_connectors:1-350942-0
Connections:
- no-connect marks 60 -> 62
Changed lines of the file:
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@@
+	)
+	(no_connect
+		(at 179.07 175.26)
 	)
 	(no_connect
@@
 	(no_connect
 		(at 300.99 149.86)
+	)
+	(no_connect
+		(at 179.07 177.8)
 	)
 	(no_connect
@@
 					(unit 1)
 				)
+			)
+		)
+	)
+	(symbol
+		(lib_id "2s_connectors:1-350942-0")
+		(at 179.07 177.8 180)
+		(unit 1)
+		(exclude_from_sim no)
+		(in_bom yes)
+		(on_board yes)
+		(dnp no)
+		(fields_autoplaced yes)
+		(property "Reference" "J13"
+			(at 170.18 167.64 0)
+			(effects
+				(font
+					(size 1.524 1.524)
+				)
+			)
+		)
+		(property "Value" "1-350942-0"
+			(at 170.18 170.18 0)
+			(effects
+				(font
+					(size 1.524 1.524)
+				)
+			)
+		)
+		(property "Footprint" "2s_connectors:CONN_1-350942-0_TYC"
+			(at 179.07 177.8 0)
+			(effects
+				(font
+					(size 1.27 1.27)
+					(italic yes)
+				)
+				(hide yes)
+			)
+		)
+		(property "Datasheet" "1-350942-0"
+			(at 179.07 177.8 0)
+			(effects
+				(font
+					(size 1.27 1.27)
+					(italic yes)
+				)
+				(hide yes)
+			)
+		)
+		(property "Description" "CONN HEADER R/A 2POS 6.35MM"
+			(at 179.07 177.8 0)
+			(effects
+				(font
+					(size 1.27 1.27)
+				)
+				(hide yes)
+			)
+		)
+		(property "Manufacturer" "TE Connectivity AMP Connectors"
+			(at 179.07 177.8 0)
+			(effects
+				(font
+					(size 1.27 1.27)
+				)
+				(hide yes)
+			)
+		)
+		(property "MPN" "1-350942-0"
+			(at 179.07 177.8 0)
+			(effects
+				(font
+					(size 1.27 1.27)
+				)
+				(hide yes)
+			)
+		)
+		(pin "1"
+		)
+		(pin "2"
+		)
+		(instances
+			(project ""
+				(path "/f48a671c-1542-4fb2-ac88-d921c6d4416a"
+					(reference "J13")
+					(unit 1)
+				)
