File: connector_board.kicad_pcb (KiCad board)
At the start: 2 copper layers, 40 x 22.5 mm, 2 parts, among them J1 Screw Terminal Block 5.00 mm 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

Commit message: feat: add connectors
Parts:
- removed R1: 47k_0805, Resistor_SMD:R_0805_2012Metric
- added H1: MountingHole, MountingHole:MountingHole_3.2mm_M3_Pad, F.Cu at (78.0, 91.0)
- added H2: MountingHole, MountingHole:MountingHole_3.2mm_M3_Pad, F.Cu at (174.0, 91.0)
- added H3: MountingHole, MountingHole:MountingHole_3.2mm_M3_Pad, F.Cu at (174.0, 37.0)
- added H4: MountingHole, MountingHole:MountingHole_3.2mm_M3_Pad, F.Cu at (78.0, 37.0)
- added J10: Screw Terminal Block 3.50 mm 2 pol, 2s_connectors:TerminalBlock_4Ucon_1x02_P3.50mm_Horizontal, F.Cu at (173.8, 68.8)
- added J11: 2s-tc2030-NL, Connector:Tag-Connect_TC2030-IDC-NL_2x03_P1.27mm_Vertical, F.Cu at (118.2, 48.9)
- added J12: TC2050 With UART NL, Connector:Tag-Connect_TC2050-IDC-NL_2x05_P1.27mm_Vertical, F.Cu at (91.0, 48.4)
- added J2: 2s_cortex-m-10-pin, 2s_connectors:PinHeader_2x5_P1.27_SMD, F.Cu at (147.7, 47.0)
- added J3: 2s-tc2030, Connector:Tag-Connect_TC2030-IDC-FP_2x03_P1.27mm_Vertical, F.Cu at (130.0, 47.1)
- added J4: 2s_cortex-m-10-pin, Connector:Tag-Connect_TC2050-IDC-FP_2x05_P1.27mm_Vertical, F.Cu at (106.5, 47.1)
- added J5: 1757242, Connector_Phoenix_MSTB:PhoenixContact_MSTBA_2,5_2-G-5,08_1x02_P5.08mm_Horizontal, F.Cu at (167.2, 51.0)
- added J6: S3B-ZR-SM4A-TF, 2s_connectors:JST_ZH_B3B-ZR-SM4-TF_1x03-1MP_P1.50mm_Vertical, F.Cu at (135.0, 91.0)
- added J7: JST S3B-XH-A, Connector_JST:JST_XH_S3B-XH-A_1x03_P2.50mm_Horizontal, F.Cu at (94.5, 85.1)
- added J8: JST S3B-PH-K-S, Connector_JST:JST_PH_S3B-PH-K_1x03_P2.00mm_Horizontal, F.Cu at (113.5, 88.0)
- added J9: JST SM03B-SRSS-TB, 2s_connectors:JST_SH_SM03B-SRSS-TB_1x03-1MP_P1.00mm_Horizontal, F.Cu at (153.5, 91.5)
- moved J1 37.2 mm to (173.5, 82.2), turned to 90 degrees
Connections:
- J1 pad 1: GND -> unconnected-(J1-Pin_1-Pad1)
- J1 pad 2: Net-(J1-Pin_2) -> unconnected-(J1-Pin_2-Pad2)
Routing:
- net GND: track 17.5 -> 0.00 mm
- net Net-(J1-Pin_2): track 17.3 -> 0.00 mm
Other:
- board size 40 x 22.5 mm -> 104 x 62 mm
- board text added: "Contact: SPH-002T-P0.5L (28-24 AWG)"
- board text added: "Contact: SSH-003T-P0.2-H (32-28 AWG)"
- board text added: "Contact: SXH-001T-P0.6 (28-22 AWG)"
- board text added: "Contact: SZH-002T-P0.5 (28-26 AWG)"
- board text added: "Housing: PHR-3"
- board text added: "Housing: SHR-03V-S"
- board text added: "Housing: XHP-3"
- board text added: "Housing: ZHR-3"
- board text added: "JST"
- board text added: "PH (2.00 mm)"
- board text added: "Phoenix Contact 1751248 3.50 mm"
- board text added: "Phoenix Contact 1757242 5.08 mm Plug: 1757019"
- board text added: "S3B-PH-K-S"
- board text added: "S3B-XH-A"
- board text added: "S3B-ZR-SM4A-TF"
- board text added: "SH (1.00 mm)"
- board text added: "SM03B-SRSS-TB"
- board text added: "Samtec Inc. FTSH-105-01-F-DV-K"
- board text added: "TC2030"
- board text added: "TC2030 NL"
- board text added: "TC2050"
- board text added: "TC2050 NL"
- board text added: "TE Connectivity 282836-2 5.00 mm"
- board text added: "Tag Connect"
- board text added: "XH (2.50 mm)"
- board text added: "ZH (1.50 mm)"

Commit message: feat: even more connectors
BREAKING CHANGE:
Parts:
- added J13: 1-350942-0, 2s_connectors:CONN_1-350942-0_TYC, F.Cu at (73.7, 70.7)
- moved H1 16.0 mm to (62.0, 91.0)
- moved H4 16.0 mm to (62.0, 37.0)
- moved J2 1.62 mm to (147.0, 45.5)
- moved J11 1.52 mm to (116.7, 49.1)
- moved J12 1.52 mm to (89.5, 48.6)
- moved J3 1.52 mm to (128.5, 47.4)
- moved J4 1.52 mm to (105.0, 47.4)
Other:
- board size 104 x 62 mm -> 120 x 62 mm
- board text added: "TE Connectivity 1-350942-0 Housing: 1586856-1 Contacts: 350851-1"

Commit message: fix: small improvements I guess
Parts:
- moved J11 5.94 mm to (111.2, 46.9)
- moved J12 5.94 mm to (84.0, 46.4)
- moved J3 5.94 mm to (123.0, 45.1)
- moved J4 5.94 mm to (99.5, 45.1)
- moved J10 5.41 mm to (170.8, 64.2)
- moved J2 4.72 mm to (143.5, 42.5)
- moved H2 4.61 mm to (169.5, 90.0)
- moved H3 4.47 mm to (170.0, 35.0)
- moved J1 4.05 mm to (170.5, 79.5)
- moved J6 4.00 mm to (131.0, 91.0)
- moved J7 4.00 mm to (90.5, 85.1)
- moved J8 4.00 mm to (109.5, 88.0)
- moved J9 4.00 mm to (149.5, 91.5)
- moved J13 3.21 mm to (70.5, 70.2)
- moved H4 2.83 mm to (60.0, 35.0)
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Other:
- board size 120 x 62 mm -> 120 x 65 mm
